File: Digit.sch (KiCad schematic (older format))
At the start: 4 parts, among them U201 74HC595, U202 ULN2803A

Commit message: Update packages
Parts:
- C201: footprint (none) -> Capacitors_SMD:C_0805_HandSoldering
- U201: footprint (none) -> SOIC-16_3.9x9.9mm_Pitch1.27mm
- U202: footprint (none) -> Housings_SOIC:SOIC-18W_7.5x11.6mm_Pitch1.27mm
Changed lines of the file:
@@
 F 0 "U201" H 5725 4425 50  0000 C CNN
 F 1 "74HC595" H 5825 4325 50  0000 C CNN
-F 2 "" H 5575 3725 50  0001 C CNN
+F 2 "SOIC-16_3.9x9.9mm_Pitch1.27mm" H 5575 3725 50  0001 C CNN
 F 3 "http://www.ti.com/lit/ds/symlink/sn74hc595.pdf" H 5575 3725 50  0001 C CNN
 	1    5575 3725
@@
 F 0 "U202" H 6900 4092 50  0000 C CNN
 F 1 "ULN2803A" H 6900 4001 50  0000 C CNN
-F 2 "" H 6950 2875 50  0001 L CNN
+F 2 "Housings_SOIC:SOIC-18W_7.5x11.6mm_Pitch1.27mm" H 6950 2875 50  0001 L CNN
 F 3 "http://www.ti.com/lit/ds/symlink/uln2803a.pdf" H 7000 3325 50  0001 C CNN
 	1    6900 3525
@@
 AR Path="/5D129954/5D108155" Ref="#PWR0402"  Part="1"
 AR Path="/5D12995C/5D108155" Ref="#PWR0502"  Part="1"
-F 0 "#PWR0202" H 5575 4275 50  0001 C CNN
+F 0 "#PWR0502" H 5575 4275 50  0001 C CNN
 F 1 "GND" H 5580 4352 50  0000 C CNN
 F 2 "" H 5575 4525 50  0001 C CNN
@@
 AR Path="/5D129954/5D108485" Ref="#PWR0403"  Part="1"
 AR Path="/5D12995C/5D108485" Ref="#PWR0503"  Part="1"
-F 0 "#PWR0203" H 6100 2475 50  0001 C CNN
+F 0 "#PWR0503" H 6100 2475 50  0001 C CNN
 F 1 "GND" V 6105 2597 50  0000 R CNN
 F 2 "" H 6100 2725 50  0001 C CNN
@@
 AR Path="/5D129954/5D109B6F" Ref="#PWR0405"  Part="1"
 AR Path="/5D12995C/5D109B6F" Ref="#PWR0505"  Part="1"
-F 0 "#PWR0205" H 7600 2350 50  0001 C CNN
+F 0 "#PWR0505" H 7600 2350 50  0001 C CNN
 F 1 "VD" H 7550 2650 50  0000 L CNN
 F 2 "" H 7600 2500 50  0001 C CNN
@@
 AR Path="/5D129954/5D10C645" Ref="#PWR0401"  Part="1"
 AR Path="/5D12995C/5D10C645" Ref="#PWR0501"  Part="1"
-F 0 "#PWR0201" H 5575 2350 50  0001 C CNN
+F 0 "#PWR0501" H 5575 2350 50  0001 C CNN
 F 1 "VCC" H 5592 2673 50  0000 C CNN
 F 2 "" H 5575 2500 50  0001 C CNN
@@
 F 0 "C201" V 5671 2725 50  0000 C CNN
 F 1 "0μ1" V 5762 2725 50  0000 C CNN
-F 2 "" H 5900 2725 50  0001 C CNN
+F 2 "Capacitors_SMD:C_0805_HandSoldering" H 5900 2725 50  0001 C CNN
 F 3 "~" H 5900 2725 50  0001 C CNN
 	1    5900 2725
@@
 AR Path="/5D129954/5D10757C" Ref="#PWR0404"  Part="1"
 AR Path="/5D12995C/5D10757C" Ref="#PWR0504"  Part="1"
-F 0 "#PWR0204" H 6900 4275 50  0001 C CNN
+F 0 "#PWR0504" H 6900 4275 50  0001 C CNN
 F 1 "GND" H 6905 4352 50  0000 C CNN
 F 2 "" H 6900 4525 50  0001 C CNN
