File: Digit.sch (KiCad schematic (older format))
At the start: 4 parts, among them U201 74HC595, U202 ULN2803A

Commit message: adding atmega328p-au
Connections:
- net labels added: CLOCK, DIN, DOUT, LATCH, ~RESET
- net labels removed: CASC, RCLK, SER, SRCLK, ~SRCLR
Changed lines of the file:
@@
 AR Path="/5D129954/5D1035D1" Ref="DS401"  Part="1"
 AR Path="/5D12995C/5D1035D1" Ref="DS501"  Part="1"
-F 0 "DS201" V 8204 3447 50  0000 R CNN
+F 0 "DS501" V 8204 3447 50  0000 R CNN
 F 1 "IV-9" V 8295 3447 50  0000 R CNN
 F 2 "Own:IV-9" H 8250 3225 50  0001 C CNN
@@
 AR Path="/5D129954/5D1035FB" Ref="U402"  Part="1"
 AR Path="/5D12995C/5D1035FB" Ref="U502"  Part="1"
-F 0 "U202" H 6900 4392 50  0000 C CNN
+F 0 "U502" H 6900 4392 50  0000 C CNN
 F 1 "ULN2803A" H 6900 4301 50  0000 C CNN
 F 2 "Housings_SOIC:SOIC-18W_7.5x11.6mm_Pitch1.27mm" H 6950 3175 50  0001 L CNN
@@
 3V15
 Text HLabel 6100 4225 2    50   Output ~ 0
-CASC
+DOUT
 Wire Wire Line
 	5975 4225 6100 4225
@@
 AR Path="/5D129954/5D108155" Ref="#PWR0402"  Part="1"
 AR Path="/5D12995C/5D108155" Ref="#PWR0502"  Part="1"
-F 0 "#PWR0202" H 5575 4275 50  0001 C CNN
+F 0 "#PWR0502" H 5575 4275 50  0001 C CNN
 F 1 "GND" H 5580 4352 50  0000 C CNN
 F 2 "" H 5575 4525 50  0001 C CNN
@@
 AR Path="/5D129954/5D108485" Ref="#PWR0403"  Part="1"
 AR Path="/5D12995C/5D108485" Ref="#PWR0503"  Part="1"
-F 0 "#PWR0203" H 6100 2475 50  0001 C CNN
+F 0 "#PWR0503" H 6100 2475 50  0001 C CNN
 F 1 "GND" V 6105 2597 50  0000 R CNN
 F 2 "" H 6100 2725 50  0001 C CNN
@@
 AR Path="/5D129954/5D109B6F" Ref="#PWR0405"  Part="1"
 AR Path="/5D12995C/5D109B6F" Ref="#PWR0505"  Part="1"
-F 0 "#PWR0205" H 7600 4700 50  0001 C CNN
+F 0 "#PWR0505" H 7600 4700 50  0001 C CNN
 F 1 "VD" H 7550 5000 50  0000 L CNN
 F 2 "" H 7600 4850 50  0001 C CNN
@@
 AR Path="/5D129954/5D10C645" Ref="#PWR0401"  Part="1"
 AR Path="/5D12995C/5D10C645" Ref="#PWR0501"  Part="1"
-F 0 "#PWR0201" H 5575 2350 50  0001 C CNN
+F 0 "#PWR0501" H 5575 2350 50  0001 C CNN
 F 1 "VCC" H 5592 2673 50  0000 C CNN
 F 2 "" H 5575 2500 50  0001 C CNN
@@
 AR Path="/5D129954/5D10D50F" Ref="C401"  Part="1"
 AR Path="/5D12995C/5D10D50F" Ref="C501"  Part="1"
-F 0 "C201" V 5671 2725 50  0000 C CNN
+F 0 "C501" V 5671 2725 50  0000 C CNN
 F 1 "0μ1" V 5762 2725 50  0000 C CNN
 F 2 "Capacitors_SMD:C_0805_HandSoldering" H 5900 2725 50  0001 C CNN
@@
 AR Path="/5D129954/5D10757C" Ref="#PWR0404"  Part="1"
 AR Path="/5D12995C/5D10757C" Ref="#PWR0504"  Part="1"
-F 0 "#PWR0204" H 6900 2575 50  0001 C CNN
+F 0 "#PWR0504" H 6900 2575 50  0001 C CNN
 F 1 "GND" H 6905 2652 50  0000 C CNN
 F 2 "" H 6900 2825 50  0001 C CNN
@@
 AR Path="/5D129954/5D1035CB" Ref="U401"  Part="1"
 AR Path="/5D12995C/5D1035CB" Ref="U501"  Part="1"
-F 0 "U201" H 5725 4425 50  0000 C CNN
+F 0 "U501" H 5725 4425 50  0000 C CNN
 F 1 "74HC595" H 5825 4325 50  0000 C CNN
 F 2 "SOIC-16_3.9x9.9mm_Pitch1.27mm" H 5575 3725 50  0001 C CNN
@@
 ~OE
 Text HLabel 4625 3825 0    50   Input ~ 0
-RCLK
+LATCH
 Text HLabel 4625 3625 0    50   Input ~ 0
-~SRCLR
+~RESET
 Text HLabel 4625 3525 0    50   Input ~ 0
-SRCLK
+CLOCK
 Text HLabel 4625 3325 0    50   Input ~ 0
-SER
+DIN
 $EndSCHEMATC
