File: Numiclock.sch (KiCad schematic (older format))
At the start: 6 parts

Commit message: Rearrange partial circuit
Parts:
- gave numbers to parts that had none: 6
Connections:
- net labels added: 3V15, 5V, GND
- wire segments 48 -> 34
Other:
- moved on the sheet: R1, R2, U1, U2, U3
Changed lines of the file:
@@
 $EndDescr
 $Comp
-L Regulator_Linear:AMS1117 U?
+L Regulator_Linear:AMS1117 U1
 U 1 1 5D0F79FB
-P 2775 1275
-F 0 "U?" H 2775 1517 50  0000 C CNN
-F 1 "AMS1117" H 2775 1426 50  0000 C CNN
-F 2 "Package_TO_SOT_SMD:SOT-223-3_TabPin2" H 2775 1475 50  0001 C CNN
-F 3 "http://www.advanced-monolithic.com/pdf/ds1117.pdf" H 2875 1025 50  0001 C CNN
-	1    2775 1275
+P 6550 1275
+F 0 "U1" H 6550 1517 50  0000 C CNN
+F 1 "AMS1117" H 6550 1426 50  0000 C CNN
+F 2 "Package_TO_SOT_SMD:SOT-223-3_TabPin2" H 6550 1475 50  0001 C CNN
+F 3 "http://www.advanced-monolithic.com/pdf/ds1117.pdf" H 6650 1025 50  0001 C CNN
+	1    6550 1275
 	1    0    0    -1
 $EndComp
 $Comp
-L Transistor_Array:ULN2803A U?
-U 1 1 5D0F8877
-P 5450 2975
-F 0 "U?" H 5450 3542 50  0000 C CNN
-F 1 "ULN2803A" H 5450 3451 50  0000 C CNN
-F 2 "" H 5500 2325 50  0001 L CNN
-F 3 "http://www.ti.com/lit/ds/symlink/uln2803a.pdf" H 5550 2775 50  0001 C CNN
-	1    5450 2975
+L Device:R_Small R1
+U 1 1 5D0FABD1
+P 6825 1675
+F 0 "R1" H 6884 1721 50  0000 L CNN
+F 1 "100" H 6884 1630 50  0000 L CNN
+F 2 "" H 6825 1675 50  0001 C CNN
+F 3 "~" H 6825 1675 50  0001 C CNN
+	1    6825 1675
+	0    -1   -1   0
+$EndComp
+$Comp
+L Device:R_Small R2
+U 1 1 5D0FB650
+P 6550 1950
+F 0 "R2" H 6609 1996 50  0000 L CNN
+F 1 "150" H 6609 1905 50  0000 L CNN
+F 2 "" H 6550 1950 50  0001 C CNN
+F 3 "~" H 6550 1950 50  0001 C CNN
+	1    6550 1950
+	1    0    0    -1
+$EndComp
+Wire Wire Line
+	6550 1575 6550 1675
+$Comp
+L 74xx:74HC595 U2
+U 1 1 5D0FC59B
+P 4925 3175
+F 0 "U2" H 4925 3956 50  0000 C CNN
+F 1 "74HC595" H 4925 3865 50  0000 C CNN
+F 2 "" H 4925 3175 50  0001 C CNN
+F 3 "http://www.ti.com/lit/ds/symlink/sn74hc595.pdf" H 4925 3175 50  0001 C CNN
+	1    4925 3175
 	1    0    0    -1
 $EndComp
 $Comp
-L Device:R_Small R?
-U 1 1 5D0FABD1
-P 3200 1500
-F 0 "R?" H 3259 1546 50  0000 L CNN
-F 1 "100" H 3259 1455 50  0000 L CNN
-F 2 "" H 3200 1500 50  0001 C CNN
-F 3 "~" H 3200 1500 50  0001 C CNN
-	1    3200 1500
-	1    0    0    -1
-$EndComp
-$Comp
-L Device:R_Small R?
-U 1 1 5D0FB650
-P 3200 2025
-F 0 "R?" H 3259 2071 50  0000 L CNN
-F 1 "150" H 3259 1980 50  0000 L CNN
-F 2 "" H 3200 2025 50  0001 C CNN
-F 3 "~" H 3200 2025 50  0001 C CNN
-	1    3200 2025
-	1    0    0    -1
-$EndComp
-Wire Wire Line
-	2775 1575 2775 1750
-Wire Wire Line
-	2775 1750 3200 1750
-Wire Wire Line
-	3200 1750 3200 1600
-Wire Wire Line
-	3200 1400 3200 1275
-Wire Wire Line
-	3200 1275 3075 1275
-Wire Wire Line
-	3200 1750 3200 1925
-Connection ~ 3200 1750
-$Comp
-L 74xx:74HC595 U?
-U 1 1 5D0FC59B
-P 4075 3175
-F 0 "U?" H 4075 3956 50  0000 C CNN
-F 1 "74HC595" H 4075 3865 50  0000 C CNN
-F 2 "" H 4075 3175 50  0001 C CNN
-F 3 "http://www.ti.com/lit/ds/symlink/sn74hc595.pdf" H 4075 3175 50  0001 C CNN
-	1    4075 3175
-	1    0    0    -1
-$EndComp
-Wire Wire Line
-	4475 2775 5050 2775
-Wire Wire Line
-	4475 2875 5050 2875
-Wire Wire Line
-	4475 2975 5050 2975
-Wire Wire Line
-	4475 3075 5050 3075
-Wire Wire Line
-	4475 3175 5050 3175
-Wire Wire Line
-	4475 3275 5050 3275
-Wire Wire Line
-	4475 3375 5050 3375
-Wire Wire Line
-	4475 3475 5050 3475
-$Comp
-L Eigene~Bauteile:IV-9 DS?
+L Eigene~Bauteile:IV-9 DS1
 U 1 1 5D0F85FE
-P 7375 3125
-F 0 "DS?" V 7329 2847 50  0000 R CNN
-F 1 "IV-9" V 7420 2847 50  0000 R CNN
-F 2 "" H 7375 2625 50  0001 C CNN
-F 3 "" H 7375 3275 50  0001 C CNN
-	1    7375 3125
+P 7750 3075
+F 0 "DS1" V 7704 2797 50  0000 R CNN
+F 1 "IV-9" V 7795 2797 50  0000 R CNN
+F 2 "" H 7750 2575 50  0001 C CNN
+F 3 "" H 7750 3225 50  0001 C CNN
+	1    7750 3075
 	0    -1   1    0
 $EndComp
 Wire Wire Line
-	6925 3525 6400 3525
+	6350 2675 7100 2675
 Wire Wire Line
-	6400 3175 5850 3175
+	7100 2675 7300 2675
+Connection ~ 7100 2675
 Wire Wire Line
-	6925 3225 6500 3225
+	6550 1850 6550 1675
 Wire Wire Line
-	6500 3225 6500 3275
+	7100 1275 7100 1675
 Wire Wire Line
-	6500 3275 5850 3275
+	6350 2775 7300 2775
 Wire Wire Line
-	6925 3325 6500 3325
+	6350 2875 7300 2875
 Wire Wire Line
-	6500 3325 6500 3375
+	7300 2975 6350 2975
 Wire Wire Line
-	6500 3375 5850 3375
+	6350 3075 7300 3075
 Wire Wire Line
-	6925 2825 6450 2825
+	7300 3175 6350 3175
 Wire Wire Line
-	6450 2825 6450 3475
+	6350 3275 7300 3275
 Wire Wire Line
-	6450 3475 5850 3475
+	6350 3375 7300 3375
 Wire Wire Line
-	5850 2675 6400 2675
+	6350 3475 7300 3475
 Wire Wire Line
-	6400 2675 6400 2725
+	5325 3475 5550 3475
 Wire Wire Line
-	6400 2725 6925 2725
+	5325 2775 5550 2775
 Wire Wire Line
-	6400 3525 6400 3175
+	5325 2875 5550 2875
 Wire Wire Line
-	6350 3075 5850 3075
+	5550 2975 5325 2975
 Wire Wire Line
-	6925 3425 6350 3425
+	5325 3075 5550 3075
 Wire Wire Line
-	6350 3425 6350 3075
+	5550 3175 5325 3175
 Wire Wire Line
-	6350 2975 5850 2975
+	5325 3275 5550 3275
 Wire Wire Line
-	6925 3025 6350 3025
+	5325 3375 5550 3375
 Wire Wire Line
-	6350 3025 6350 2975
+	4925 3875 4925 4225
+Connection ~ 4925 4225
 Wire Wire Line
-	6350 2875 5850 2875
+	4925 4225 5950 4225
+Connection ~ 6550 1675
 Wire Wire Line
-	6925 2925 6350 2925
+	6550 1675 6725 1675
 Wire Wire Line
-	6350 2925 6350 2875
+	6850 1275 7100 1275
 Wire Wire Line
-	6400 2775 5850 2775
+	7100 1675 6925 1675
 Wire Wire Line
-	6925 3125 6400 3125
+	2225 4225 4925 4225
 Wire Wire Line
-	6400 3125 6400 2775
+	6250 1275 4925 1275
+Connection ~ 7100 1675
 Wire Wire Line
-	6400 2675 6400 1275
+	7100 1675 7100 2675
 Wire Wire Line
-	6400 1275 3200 1275
-Connection ~ 6400 2675
-Connection ~ 3200 1275
+	4925 2575 4925 1275
+Connection ~ 4925 1275
 Wire Wire Line
-	5450 3675 5450 4225
+	4925 1275 2225 1275
 Wire Wire Line
-	5450 4225 4075 4225
+	6550 2050 6550 4225
+$Comp
+L Transistor_Array:ULN2803A U3
+U 1 1 5D0F8877
+P 5950 2975
+F 0 "U3" H 5950 3542 50  0000 C CNN
+F 1 "ULN2803A" H 5950 3451 50  0000 C CNN
+F 2 "" H 6000 2325 50  0001 L CNN
+F 3 "http://www.ti.com/lit/ds/symlink/uln2803a.pdf" H 6050 2775 50  0001 C CNN
+	1    5950 2975
+	1    0    0    -1
+$EndComp
+Connection ~ 5950 4225
 Wire Wire Line
-	4075 4225 4075 3875
+	5950 4225 6550 4225
+Text Label 5500 1275 0    50   ~ 0
+5V
+Text Label 7100 1275 0    50   ~ 0
+3V15
+Text Label 6550 4225 0    50   ~ 0
+GND
 Wire Wire Line
-	3200 2125 3200 4225
-Wire Wire Line
-	3200 4225 4075 4225
-Connection ~ 4075 4225
+	5950 3675 5950 4225
 $EndSCHEMATC

Commit message: Using hierarchical schematics for each digit unit; include IV-9 footprint
Parts:
- removed DS1: IV-9, symbol Eigene~Bauteile:IV-9
- removed U2: 74HC595, symbol 74xx:74HC595
- removed U3: ULN2803A, symbol Transistor_Array:ULN2803A
- added J101: Barrel_Jack_Switch, symbol Connector:Barrel_Jack_Switch
- added R103, R104: 10k, symbol Device:R_Small
- added U102: DCF1, symbol Eigene~Bauteile:DCF1
- renumbered R2 to R101, R1 to R102, U1 to U101
Connections:
- net labels added: VCC, VD
- wire segments 34 -> 69
- no-connect marks 0 -> 2
Other:
- moved on the sheet: R101, R102, U101

Commit message: Update packages
Parts:
- J101: footprint (none) -> Connectors:BARREL_JACK
- R101, R102, R103, R104: footprint (none) -> Resistors_SMD:R_0805_HandSoldering
- U101: footprint Package_TO_SOT_SMD:SOT-223-3_TabPin2 -> TO_SOT_Packages_SMD:SOT-223
- U102: footprint (none) -> Own:DCF1
Changed lines of the file:
@@
 F 0 "U101" H 10025 1317 50  0000 C CNN
 F 1 "AMS1117" H 10025 1226 50  0000 C CNN
-F 2 "Package_TO_SOT_SMD:SOT-223-3_TabPin2" H 10025 1275 50  0001 C CNN
+F 2 "TO_SOT_Packages_SMD:SOT-223" H 10025 1275 50  0001 C CNN
 F 3 "http://www.advanced-monolithic.com/pdf/ds1117.pdf" H 10125 825 50  0001 C CNN
 	1    10025 1075
@@
 F 0 "R102" H 10459 1321 50  0000 L CNN
 F 1 "100" H 10459 1230 50  0000 L CNN
-F 2 "" H 10400 1275 50  0001 C CNN
+F 2 "Resistors_SMD:R_0805_HandSoldering" H 10400 1275 50  0001 C CNN
 F 3 "~" H 10400 1275 50  0001 C CNN
 	1    10400 1275
@@
 F 0 "R101" H 10459 1721 50  0000 L CNN
 F 1 "150" H 10459 1630 50  0000 L CNN
-F 2 "" H 10400 1675 50  0001 C CNN
+F 2 "Resistors_SMD:R_0805_HandSoldering" H 10400 1675 50  0001 C CNN
 F 3 "~" H 10400 1675 50  0001 C CNN
 	1    10400 1675
@@
 F 0 "R103" H 5234 5096 50  0000 L CNN
 F 1 "10k" H 5234 5005 50  0000 L CNN
-F 2 "" H 5175 5050 50  0001 C CNN
+F 2 "Resistors_SMD:R_0805_HandSoldering" H 5175 5050 50  0001 C CNN
 F 3 "~" H 5175 5050 50  0001 C CNN
 	1    5175 5050
@@
 F 0 "R104" H 5534 5096 50  0000 L CNN
 F 1 "10k" H 5534 5005 50  0000 L CNN
-F 2 "" H 5475 5050 50  0001 C CNN
+F 2 "Resistors_SMD:R_0805_HandSoldering" H 5475 5050 50  0001 C CNN
 F 3 "~" H 5475 5050 50  0001 C CNN
 	1    5475 5050
@@
 F 0 "U102" H 7653 2578 60  0000 L CNN
 F 1 "DCF1" H 7653 2472 60  0000 L CNN
-F 2 "" H 7475 2350 60  0001 C CNN
+F 2 "Own:DCF1" H 7475 2350 60  0001 C CNN
 F 3 "" H 7475 2350 60  0001 C CNN
 	1    7275 2550
@@
 F 0 "J101" H 1357 1667 50  0000 C CNN
 F 1 "Barrel_Jack_Switch" H 1357 1576 50  0000 C CNN
-F 2 "" H 1350 1310 50  0001 C CNN
+F 2 "Connectors:BARREL_JACK" H 1350 1310 50  0001 C CNN
 F 3 "~" H 1350 1310 50  0001 C CNN
 	1    1300 1350

Commit message: adding atmega328p-au
Parts:
- added C101, C102, C103, C104: 0μ1, Capacitors_SMD:C_0805_HandSoldering, symbol Device:C_Small
- added C105, C106: 22p, Capacitors_SMD:C_0805_HandSoldering, symbol Device:C_Small
- added ISP101: Conn_02x03_Odd_Even, Own:Pin_Header_Straight_Shrouded_2x03_Pitch2.54mm_ConvNumbering, symbol Connector_Generic:Conn_02x03_Odd_Even
- added R105, R106: 10k, Resistors_SMD:R_0805_HandSoldering, symbol Device:R_Small
- added SERPRG101: Conn_01x06, Socket_Strips:Socket_Strip_Straight_1x06_Pitch2.54mm, symbol Connector_Generic:Conn_01x06
- added U102: ATmega328P-AU, Housings_QFP:TQFP-32_7x7mm_Pitch0.8mm, symbol MCU_Microchip_ATmega:ATmega328P-AU
- added Y101: 16M, Crystals:Crystal_SMD_3225-4pin_3.2x2.5mm_HandSoldering, symbol Device:Crystal_GND24_Small
- renumbered U102 to DCF1
Connections:
- net labels added: MISO, MOSI, PR_CTS, PR_DTR, PR_RX, PR_TX, RXD, SCK, TXD, XTAL1, XTAL2, ~SS
- wire segments 69 -> 132
- no-connect marks 2 -> 17
Other:
- moved on the sheet: J101
